File: drink_water_pcb/drink_water/drink_water.kicad_pcb (KiCad board)
At the start: 2 copper layers, 42 x 116 mm, 47 parts, among them J1 Conn_01x04, J2 USB_C_Receptacle_USB2.0_16P, J3 Conn_01x02, J4 Conn_01x02, Q1 FS8205, SW1 SW_SPDT, U1 ESP32-C3-WROOM-02, U2 USBLC6-2SC6, U3 TP4056, U4 DW01A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

Commit message: Initial layout, pre-route
Parts:
- added D4: MBRS130LT3, Diode_SMD:D_SMB, F.Cu at (111.0, 117.8)
- added Q2: AO3401A, Package_TO_SOT_SMD:SOT-23, F.Cu at (110.8, 128.1)
- added R12: 10k, Resistor_SMD:R_0402_1005Metric, F.Cu at (111.2, 124.2)
- moved C7 3.41 mm to (115.4, 122.3)
- moved C5 3.02 mm to (121.3, 125.1)
- moved C6 3.02 mm to (123.0, 116.8)
- moved Q1 3.02 mm to (115.6, 118.1)
- moved R10 3.02 mm to (118.8, 114.8)
- moved R8 3.02 mm to (121.3, 127.6)
- moved R9 3.02 mm to (123.0, 118.8)
- moved U4 3.02 mm to (120.3, 118.1)
- moved U3 3.02 mm to (116.8, 126.4)
- moved TP2 2.81 mm to (127.5, 129.0)
- moved TP1 2.80 mm to (124.8, 129.0)
Connections:
- C7 pad 1: VCC -> +BATT
- J3 pad 2: VCC -> +BATT
- U3 pad 5: VCC -> +BATT

Commit message: Initial version of PCB design
Parts:
- moved J1 36.6 mm to (140.6, 123.7), turned to -90 degrees
- moved J2 35.1 mm to (106.0, 134.6), turned to -90 degrees
- moved R4 31.1 mm to (107.6, 141.0), turned to -90 degrees
- moved C4 22.2 mm to (112.0, 130.6), turned to 90 degrees
- moved R5 20.6 mm to (112.9, 132.1), turned to 0 degrees
- moved U2 20.3 mm to (113.9, 134.6), turned to 0 degrees
- moved TP1 19.1 mm to (131.8, 111.2)
- moved TP2 17.9 mm to (129.0, 111.2)
- moved C11 4.67 mm to (123.4, 132.0), turned to 180 degrees
- moved C12 4.58 mm to (120.6, 134.1), turned to -90 degrees
- moved J4 2.85 mm to (139.4, 142.0)
- moved U3 2.41 mm to (119.2, 125.8)
- moved C5 2.41 mm to (123.6, 124.5)
- moved C6 2.41 mm to (125.4, 116.3)
- moved C7 2.41 mm to (117.8, 121.8)
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Connections:
- U1 pad 16: INT2 -> unconnected-(U1-IO2-Pad16)
- U5 pad 9: INT2 -> unconnected-(U5-INT2-Pad9)
Routing:
- net VBUS: track 0.00 -> 81.5 mm, vias 0 -> 4
- net GND: track 0.00 -> 79.7 mm, vias 0 -> 22
- net SDA: track 0.00 -> 62.2 mm, vias 0 -> 6
- net SCL: track 0.00 -> 55.3 mm, vias 0 -> 6
- net VCC: track 0.00 -> 49.0 mm, vias 0 -> 2
- net Net-(J1-Pin_3): track 0.00 -> 36.1 mm, vias 0 -> 4
- net Net-(J1-Pin_2): track 0.00 -> 35.9 mm, vias 0 -> 4
- net Net-(C8-C): track 0.00 -> 35.5 mm, vias 0 -> 1
- net Net-(C8-SHLD): track 0.00 -> 32.0 mm
- net +3V3: track 0.00 -> 31.1 mm
- net Net-(U3-CHRG#): track 0.00 -> 23.2 mm, vias 0 -> 2
- net Net-(U3-STDBY#): track 0.00 -> 22.1 mm, vias 0 -> 2
- net -BATT: track 0.00 -> 21.8 mm
- net USB_DN: track 0.00 -> 16.5 mm
- net INT1: track 0.00 -> 16.2 mm, vias 0 -> 2
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- added copper zone on F.Cu, net +3V3
- added copper zone on B.Cu, net GND
Other:
- outline, holes or cut-outs redrawn

Commit message: Shifted USB port proud of board
Parts:
- added Drink Water V0.1.0: https://github.com/heidtn/drinkmoarwater, custom_parts:https___github.com_heidtn_drinkmoarwater, B.Cu at (135.2, 109.4)
- moved J2 1.64 mm to (104.4, 134.6)
Routing:
- net VBUS: track 81.5 -> 84.8 mm
- net Net-(J2-D--PadA7): track 4.75 -> 7.47 mm
- net Net-(J2-CC2): track 6.46 -> 8.52 mm
- net Net-(J2-D+-PadA6): track 5.74 -> 7.57 mm
- net GND: track 79.7 -> 81.3 mm
- net Net-(J2-CC1): track 4.66 -> 6.22 mm
